Commit message: Add Go2-mounted observation planning

File: d1_constrained_description_20260728/urdf/d1_description.urdf (robot description, URDF)
Before this commit: robot d1_constrained_description, 10 links, 9 joints
Links:
- link Link6: geometry collision box size=0.0899313762 0.0257728751 0.02533514892; collision box size=0.130145850286 0.080071964063 0.034361989941
